Commit message: inertias updated

File: rosrider_gazebo/urdf/caretta.urdf (robot description, URDF)
Before this commit: robot caretta, 7 links, 6 joints
Links:
- link base_link: mass 2.2 -> None; geometry visual mesh filename=package://rosrider_gazebo/models/common/meshes/caretta.stl scale=0.001 0.001 0.001
- link base_scan: mass 0.2 -> None; geometry visual cylinder length=0.022 radius=0.0328
- link caster_back_link: mass 0.1 -> None; geometry visual sphere radius=0.012
- link wheel_left_link: mass 0.06 -> None; geometry visual mesh filename=package://rosrider_gazebo/models/common/meshes/wheel_left.s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 scale=0.001 0.001 0.001
- link wheel_right_link: mass 0.06 -> None; geometry visual mesh filename=package://rosrider_gazebo/models/common/meshes/wheel_right.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 scale=0.001 0.001 0.001
Joints:
- joint scan_joint: origin xyz=-0.063 0 0.052 rpy=0 0 0 -> xyz=-0.063 0 0.06975 rpy=0 0 0

File: rosrider_gazebo/urdf/sorcerer.urdf (robot description, URDF)
Before this commit: robot sorcerer, 7 links, 6 joints
Links:
- link base_link: mass 1.6 -> None; geometry visual mesh filename=package://rosrider_gazebo/models/common/meshes/sorcerer.stl scale=0.001 0.001 0.001
- link base_scan: mass 0.2 -> None; geometry visual cylinder length=0.012 radius=0.018
- link caster_back_link: mass 0.1 -> None; geometry visual sphere radius=0.0095
- link wheel_left_link: mass 0.06 -> None; geometry visual mesh filename=package://rosrider_gazebo/models/common/meshes/wheel_left.s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 scale=0.001 0.001 0.001
- link wheel_right_link: mass 0.06 -> None; geometry visual mesh filename=package://rosrider_gazebo/models/common/meshes/wheel_right.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 scale=0.001 0.001 0.001
Joints:
- joint scan_joint: origin xyz=-0.067 0 0.1154 rpy=0 0 0 -> xyz=-0.067 0 0.12 rpy=0 0 0

Commit message: minor fixes

File: rosrider_gazebo/urdf/caretta.urdf (robot description, URDF)
Before this commit: robot caretta, 7 links, 6 joints
Links:
- link caster_back_link: geometry visual sphere radius=0.01
Joints:
- joint caster_back_joint: origin xyz=-0.1454 0 -0.02225 rpy=0 0 0 -> xyz=-0.1454 0 -0.02425 rpy=0 0 0

File: rosrider_gazebo/urdf/sorcerer.urdf (robot description, URDF)
Before this commit: robot sorcerer, 7 links, 6 joints
Links:
- link caster_back_link: geometry visual sphere radius=0.01
Joints:
- joint caster_back_joint: origin xyz=-0.09 0 -0.02475 rpy=0 0 0 -> xyz=-0.09 0 -0.02425 rpy=0 0 0
