Commit message: model changes

File: rosrider_description/urdf/caretta.urdf (robot description, URDF)
Before this commit: robot sorcerer, 7 links, 6 joints
Links:
- link base_link: geometry visual mesh filename=package://rosrider_description/models/common/meshes/caretta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 scale=0.001 0.001 0.001
- link base_scan: geometry visual cylinder length=0.022 radius=0.0328
- link wheel_left_link: geometry visual mesh filename=package://rosrider_description/models/common/meshes/wheel_l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 scale=0.001 0.001 0.001
- link wheel_right_link: geometry visual mesh filename=package://rosrider_description/models/common/meshes/wheel_r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 scale=0.001 0.001 0.001
Joints:
- joint caster_back_joint: origin xyz=-0.09 0 -0.02425 rpy=0 0 0 -> xyz=-0.1454 0 -0.02425 rpy=0 0 0
- joint imu_joint: origin xyz=0.008 0 0.0884 rpy=0 0 0 -> xyz=-0.056 0.078 0.0396 rpy=0 0 0
- joint scan_joint: origin xyz=-0.067 0 0.12 rpy=0 0 0 -> xyz=-0.063 0 0.06975 rpy=0 0 0
- joint wheel_left_joint: origin xyz=0.0 0.05 0.0 rpy=-1.57 0 0 -> xyz=0.0 0.092 0.0 rpy=-1.57 0 0
- joint wheel_right_joint: origin xyz=0.0 -0.05 0.0 rpy=-1.57 0 0 -> xyz=0.0 -0.092 0.0 rpy=-1.57 0 0

File: rosrider_description/urdf/sorcerer.urdf (robot description, URDF)
Before this commit: robot caretta, 7 links, 6 joints
Links:
- link base_link: geometry visual mesh filename=package://rosrider_description/models/common/meshes/sorcere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 scale=0.001 0.001 0.001
- link base_scan: geometry visual cylinder length=0.012 radius=0.018
- link wheel_left_link: geometry visual mesh filename=package://rosrider_description/models/common/meshes/wheel_l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 scale=0.001 0.001 0.001
- link wheel_right_link: geometry visual mesh filename=package://rosrider_description/models/common/meshes/wheel_r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 scale=0.001 0.001 0.001
Joints:
- joint caster_back_joint: origin xyz=-0.1454 0 -0.02425 rpy=0 0 0 -> xyz=-0.09 0 -0.02425 rpy=0 0 0
- joint imu_joint: origin xyz=-0.056 0.078 0.0396 rpy=0 0 0 -> xyz=0.008 0 0.0884 rpy=0 0 0
- joint scan_joint: origin xyz=-0.063 0 0.06975 rpy=0 0 0 -> xyz=-0.067 0 0.12 rpy=0 0 0
- joint wheel_left_joint: origin xyz=0.0 0.092 0.0 rpy=-1.57 0 0 -> xyz=0.0 0.05 0.0 rpy=-1.57 0 0
- joint wheel_right_joint: origin xyz=0.0 -0.092 0.0 rpy=-1.57 0 0 -> xyz=0.0 -0.05 0.0 rpy=-1.57 0 0

Commit message: updates

File: rosrider_description/urdf/caretta.urdf (robot description, URDF)
Before this commit: robot caretta, 7 links, 6 joints
Links:
- link base_link: geometry visual mesh filename=package://rosrider_description/meshes/caretta.stl scale=0.001 0.001 0.001
- link wheel_left_link: geometry visual mesh filename=package://rosrider_description/meshes/wheel_left.stl scale=0.001 0.001 0.001
- link wheel_right_link: geometry visual mesh filename=package://rosrider_description/meshes/wheel_right.stl scale=0.001 0.001 0.001

File: rosrider_description/urdf/sorcerer.urdf (robot description, URDF)
Before this commit: robot sorcerer, 7 links, 6 joints
Links:
- link base_link: geometry visual mesh filename=package://rosrider_description/meshes/sorcerer.stl scale=0.001 0.001 0.001
- link wheel_left_link: geometry visual mesh filename=package://rosrider_description/meshes/wheel_left.stl scale=0.001 0.001 0.001
- link wheel_right_link: geometry visual mesh filename=package://rosrider_description/meshes/wheel_right.stl scale=0.001 0.001 0.001
